File: Schematics/cameraBoardSchematic/Camera_center.kicad_sch (KiCad schematic)
At the start: 7 parts, among them IC1 LM3940IS-3.3_NOPB

Commit message: first PCB Draft
Parts:
- removed C11: 33u, Capacitor_SMD:C_0805_2012Metric_Pad1.18x1.45mm_HandSolder, symbol Device:C
- removed C3: 1u, Capacitor_SMD:C_0805_2012Metric_Pad1.18x1.45mm_HandSolder, symbol Device:C
- removed IC1: LM3940IS-3.3_NOPB, myFootprints:TO254P1524X483-4N, symbol LM3940IS-3.3_NOPB:LM3940IS-3.3_NOPB
- removed J_BUCK_IN_A1, J_BUCK_IN_B1, J_BUCK_OUT_A1, J_BUCK_OUT_B1: ~, Capacitor_SMD:C_0805_2012Metric_Pad1.18x1.45mm_HandSolder, symbol Connector_Generic:Conn_01x02
- added C28, C29: 1u, Capacitor_SMD:C_0805_2012Metric_Pad1.18x1.45mm_HandSolder, symbol Device:C
- added C30: 47u, Capacitor_SMD:C_0805_2012Metric_Pad1.18x1.45mm_HandSolder, symbol Device:C
- added C31: .1u, Capacitor_SMD:C_0805_2012Metric_Pad1.18x1.45mm_HandSolder, symbol Device:C
- added J5: Runcam Split 4 v2, Capacitor_SMD:C_0805_2012Metric_Pad1.18x1.45mm_HandSolder, symbol Connector_Generic:Conn_01x05
- added R10: 1k, Resistor_SMD:R_0805_2012Metric_Pad1.20x1.40mm_HandSolder, symbol Device:R
- added R9: 100k, Resistor_SMD:R_0805_2012Metric_Pad1.20x1.40mm_HandSolder, symbol Device:R
- added U6: TPS22917DBVR, myFootprints:SOT95P280X145-6N, symbol TPS22917DBVR:TPS22917DBVR
Connections:
- net +3.3V: now also R9.2
- net +5V: now also C28.1, U6.1 (VIN)
- net GND: now also C28.2, C29.2, C30.2, C31.2, J5.4 (GND), R10.2, U6.2 (GND)
- new net: C29.1, C30.1, C31.1, J5.5 (VCC), U6.5 (QOD), U6.6 (VOUT)
- new net CAM_C_PWN_EN: R9.1, U6.3 (ON)
- new net CAM_UART_TX: J5.1 (RX), R10.1
