File: Schematics/cameraBoardSchematic/Camera_right.kicad_sch (KiCad schematic)
At the start: 7 parts, among them IC1 LM3940IS-3.3_NOPB

Commit message: first PCB Draft
Parts:
- removed C11: 33u, Capacitor_SMD:C_0805_2012Metric_Pad1.18x1.45mm_HandSolder, symbol Device:C
- removed C3: 1u, Capacitor_SMD:C_0805_2012Metric_Pad1.18x1.45mm_HandSolder, symbol Device:C
- removed IC1: LM3940IS-3.3_NOPB, myFootprints:TO254P1524X483-4N, symbol LM3940IS-3.3_NOPB:LM3940IS-3.3_NOPB
- removed J_BUCK_IN_A1, J_BUCK_IN_B1, J_BUCK_OUT_A1, J_BUCK_OUT_B1: ~, Capacitor_SMD:C_0805_2012Metric_Pad1.18x1.45mm_HandSolder, symbol Connector_Generic:Conn_01x02
- added C24, C25: 1u, Capacitor_SMD:C_0805_2012Metric_Pad1.18x1.45mm_HandSolder, symbol Device:C
- added C26: 47u, Capacitor_SMD:C_0805_2012Metric_Pad1.18x1.45mm_HandSolder, symbol Device:C
- added C27: .1u, Capacitor_SMD:C_0805_2012Metric_Pad1.18x1.45mm_HandSolder, symbol Device:C
- added J4: Runcam Split 4 v2, Capacitor_SMD:C_0805_2012Metric_Pad1.18x1.45mm_HandSolder, symbol Connector_Generic:Conn_01x05
- added R7: 100k, Resistor_SMD:R_0805_2012Metric_Pad1.20x1.40mm_HandSolder, symbol Device:R
- added R8: 1k, Resistor_SMD:R_0805_2012Metric_Pad1.20x1.40mm_HandSolder, symbol Device:R
- added U3: TPS22917DBVR, myFootprints:SOT95P280X145-6N, symbol TPS22917DBVR:TPS22917DBVR
Connections:
- net +3.3V: now also R7.2
- net +5V: now also C24.1, U3.1 (VIN)
- net GND: now also C24.2, C25.2, C26.2, C27.2, J4.4 (GND), R8.2, U3.2 (GND)
- new net: C25.1, C26.1, C27.1, J4.5 (VCC), U3.5 (QOD), U3.6 (VOUT)
- new net CAM_R_PWN_EN: R7.1, U3.3 (ON)
- new net CAM_UART_TX: J4.1 (RX), R8.1
