File: Schematics/cameraBoardSchematic/power.kicad_sch (KiCad schematic)
At the start: 7 parts, among them IC1 LM3940IS-3.3_NOPB

Commit message: first PCB Draft
Connections:
- net GND: no longer J_BUCK_OUT_B1.2 (Pin_2)
Changed lines of the file:
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@@
-	(wire
-		(pts
-			(xy 157.48 49.53) (xy 151.13 49.53)
-		)
-		(stroke
-			(width 0)
-			(type default)
-		)
-	)
 	(wire
 		(pts
