File: Schematics/usb_type_c_sch.kicad_sch (KiCad schematic)
At the start: 4 parts, among them J2 USB_C_Receptacle

Commit message: final design pcb
Parts:
- renumbered D1 to D4, R6 to R7, R5 to R8
Connections:
- net +5V renamed USB 5v
Changed lines of the file:
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@@
 	)
 	(junction
-		(at 147.32 67.31)
+		(at 163.83 57.15)
 		(diameter 0)
 		(color 0 0 0 0)
@@
 	)
 	(junction
+		(at 154.94 67.31)
+		(diameter 0)
+		(color 0 0 0 0)
+	)
+	(junction
 		(at 147.32 86.36)
 		(diameter 0)
@@
 	(wire
 		(pts
+			(xy 163.83 57.15) (xy 163.83 53.34)
+		)
+		(stroke
+			(width 0)
+			(type default)
+		)
+	)
+	(wire
+		(pts
 			(xy 147.32 87.63) (xy 140.97 87.63)
 		)
@@
 	(wire
 		(pts
+			(xy 163.83 57.15) (xy 165.1 57.15)
+		)
+		(stroke
+			(width 0)
+			(type default)
+		)
+	)
+	(wire
+		(pts
 			(xy 193.04 82.55) (xy 193.04 83.82)
 		)
@@
 	(wire
 		(pts
+			(xy 160.02 57.15) (xy 160.02 67.31)
+		)
+		(stroke
+			(width 0)
+			(type default)
+		)
+	)
+	(wire
+		(pts
 			(xy 147.32 81.28) (xy 147.32 82.55)
 		)
@@
 	(wire
 		(pts
-			(xy 140.97 67.31) (xy 147.32 67.31)
-		)
-		(stroke
-			(width 0)
-			(type default)
-		)
-	)
-	(wire
-		(pts
-			(xy 147.32 67.31) (xy 158.75 67.31)
+			(xy 140.97 67.31) (xy 154.94 67.31)
 		)
 		(stroke
@@
 	(wire
 		(pts
-			(xy 147.32 63.5) (xy 147.32 67.31)
-		)
-		(stroke
-			(width 0)
-			(type default)
-		)
-	)
-	(wire
-		(pts
 			(xy 158.75 86.36) (xy 158.75 78.74)
 		)
@@
 	(wire
 		(pts
+			(xy 160.02 57.15) (xy 163.83 57.15)
+		)
+		(stroke
+			(width 0)
+			(type default)
+		)
+	)
+	(wire
+		(pts
 			(xy 125.73 134.62) (xy 125.73 133.35)
 		)
@@
 	(wire
 		(pts
+			(xy 163.83 53.34) (xy 165.1 53.34)
+		)
+		(stroke
+			(width 0)
+			(type default)
+		)
+	)
+	(wire
+		(pts
 			(xy 147.32 86.36) (xy 153.67 86.36)
+		)
+		(stroke
+			(width 0)
+			(type default)
+		)
+	)
+	(wire
+		(pts
+			(xy 160.02 67.31) (xy 154.94 67.31)
 		)
 		(stroke
@@
 		)
 	)
+	(hierarchical_label "USB 5v"
+		(shape input)
+		(at 182.88 81.28 0)
+		(effects
+			(font
+				(size 1.27 1.27)
+			)
+			(justify left)
+		)
+	)
+	(hierarchical_label "USB 5v"
+		(shape input)
+		(at 165.1 57.15 0)
+		(effects
+			(font
+				(size 1.27 1.27)
+			)
+			(justify left)
+		)
+	)
 	(hierarchical_label "D+"
 		(shape input)
@@
 	(hierarchical_label "VBUS"
 		(shape input)
-		(at 147.32 63.5 90)
+		(at 165.1 53.34 0)
 		(effects
 			(font
@@
 	)
 	(symbol
-		(lib_id "power:+5V")
-		(at 182.88 81.28 270)
-		(unit 1)
-		(exclude_from_sim no)
-		(in_bom yes)
-		(on_board yes)
-		(dnp no)
-		(property "Reference" "#PWR052"
-			(at 179.07 81.28 0)
-			(effects
-				(font
-					(size 1.27 1.27)
-				)
-				(hide yes)
-			)
-		)
-		(property "Value" "+5V"
-			(at 186.69 81.2801 90)
-			(effects
-				(font
-					(size 1.27 1.27)
-				)
-				(justify left)
-			)
-		)
-		(property "Footprint" ""
-			(at 182.88 81.28 0)
-			(effects
-				(font
-					(size 1.27 1.27)
-				)
-				(hide yes)
-			)
-		)
-		(property "Datasheet" ""
-			(at 182.88 81.28 0)
-			(effects
-				(font
-					(size 1.27 1.27)
-				)
-				(hide yes)
-			)
-		)
-		(property "Description" "Power symbol creates a global label with name \"+5V\""
-			(at 182.88 81.28 0)
-			(effects
-				(font
-					(size 1.27 1.27)
-				)
-				(hide yes)
-			)
-		)
-		(pin "1"
-		)
-		(instances
-			(project ""
-				(path "/65068a32-f105-4204-b50e-234054c5a6d0/880da092-1c6b-4dcf-a509-490b22fc0ebc"
-					(reference "#PWR052")
-					(unit 1)
-				)
-			)
-		)
-	)
-	(symbol
-		(lib_id "power:+5V")
-		(at 158.75 67.31 270)
+		(lib_id "power:PWR_FLAG")
+		(at 154.94 67.31 0)
 		(unit 1)
 		(exclude_from_sim no)
@@
 		(dnp no)
 		(fields_autoplaced yes)
-		(property "Reference" "#PWR050"
+		(property "Reference" "#FLG06"
+			(at 154.94 65.405 0)
+			(effects
+				(font
+					(size 1.27 1.27)
+				)
+				(hide yes)
+			)
+		)
+		(property "Value" "PWR_FLAG"
+			(at 154.94 62.23 0)
+			(effects
+				(font
+					(size 1.27 1.27)
+				)
+			)
+		)
+		(property "Footprint" ""
 			(at 154.94 67.31 0)
 			(effects
@@
 			)
 		)
-		(property "Value" "+5V"
-			(at 162.56 67.3099 90)
-			(effects
-				(font
-					(size 1.27 1.27)
-				)
-				(justify left)
-			)
-		)
-		(property "Footprint" ""
-			(at 158.75 67.31 0)
-			(effects
-				(font
-					(size 1.27 1.27)
-				)
-				(hide yes)
-			)
-		)
-		(property "Datasheet" ""
-			(at 158.75 67.31 0)
-			(effects
-				(font
-					(size 1.27 1.27)
-				)
-				(hide yes)
-			)
-		)
-		(property "Description" "Power symbol creates a global label with name \"+5V\""
-			(at 158.75 67.31 0)
+		(property "Datasheet" "~"
+			(at 154.94 67.31 0)
+			(effects
+				(font
+					(size 1.27 1.27)
+				)
+				(hide yes)
+			)
+		)
+		(property "Description" "Special symbol for telling ERC where power comes from"
+			(at 154.94 67.31 0)
 			(effects
 				(font
@@
 			(project ""
 				(path "/65068a32-f105-4204-b50e-234054c5a6d0/880da092-1c6b-4dcf-a509-490b22fc0ebc"
-					(reference "#PWR050")
+					(reference "#FLG06")
 					(unit 1)
 				)
@@
 		(on_board yes)
 		(dnp no)
-		(property "Reference" "D1"
+		(property "Reference" "D4"
 			(at 170.18 91.44 0)
 			(effects
@@
 			(project ""
 				(path "/65068a32-f105-4204-b50e-234054c5a6d0/880da092-1c6b-4dcf-a509-490b22fc0ebc"
-					(reference "D1")
+					(reference "D4")
 					(unit 1)
 				)
@@
 		(dnp no)
 		(fields_autoplaced yes)
-		(property "Reference" "#PWR048"
+		(property "Reference" "#PWR065"
 			(at 193.04 90.17 0)
 			(effects
@@
 			(project ""
 				(path "/65068a32-f105-4204-b50e-234054c5a6d0/880da092-1c6b-4dcf-a509-490b22fc0ebc"
-					(reference "#PWR048")
+					(reference "#PWR065")
 					(unit 1)
 				)
@@
 		(on_board yes)
 		(dnp no)
-		(property "Reference" "#PWR051"
+		(property "Reference" "#PWR063"
 			(at 189.23 78.74 0)
 			(effects
@@
 			(project ""
 				(path "/65068a32-f105-4204-b50e-234054c5a6d0/880da092-1c6b-4dcf-a509-490b22fc0ebc"
-					(reference "#PWR051")
+					(reference "#PWR063")
 					(unit 1)
 				)
@@
 		(dnp no)
 		(fields_autoplaced yes)
-		(property "Reference" "#PWR047"
+		(property "Reference" "#PWR061"
 			(at 121.92 144.78 0)
 			(effects
@@
 			(project ""
 				(path "/65068a32-f105-4204-b50e-234054c5a6d0/880da092-1c6b-4dcf-a509-490b22fc0ebc"
-					(reference "#PWR047")
+					(reference "#PWR061")
 					(unit 1)
 				)
@@
 		(dnp no)
 		(fields_autoplaced yes)
-		(property "Reference" "R6"
+		(property "Reference" "R7"
 			(at 195.58 77.4699 0)
 			(effects
@@
 			(project ""
 				(path "/65068a32-f105-4204-b50e-234054c5a6d0/880da092-1c6b-4dcf-a509-490b22fc0ebc"
-					(reference "R6")
+					(reference "R7")
 					(unit 1)
 				)
@@
 		(dnp no)
 		(fields_autoplaced yes)
-		(property "Reference" "#PWR049"
+		(property "Reference" "#PWR066"
 			(at 204.47 87.63 0)
 			(effects
@@
 			(project ""
 				(path "/65068a32-f105-4204-b50e-234054c5a6d0/880da092-1c6b-4dcf-a509-490b22fc0ebc"
-					(reference "#PWR049")
+					(reference "#PWR066")
 					(unit 1)
 				)
@@
 		(dnp no)
 		(fields_autoplaced yes)
-		(property "Reference" "R5"
+		(property "Reference" "R8"
 			(at 207.01 74.9299 0)
 			(effects
@@
 			(project ""
 				(path "/65068a32-f105-4204-b50e-234054c5a6d0/880da092-1c6b-4dcf-a509-490b22fc0ebc"
-					(reference "R5")
+					(reference "R8")
 					(unit 1)
 				)
