File: Schematics/power.kicad_sch (KiCad schematic)
At the start: 10 parts, among them U2 LDL1117-3.3

Commit message: updated v2 now ready for order
Connections:
- net +3.3V: now also U2.2 (Vout); no longer U2.3 (Vout)
- net GND: now also U2.1 (GND); no longer U2.2 (GND)
- net at C16.1, D2.1 (K), D3.1 (K): now also U2.3 (Vin); no longer U2.1 (Vin)
